Commit message: 加入圆柱体并修改obs, events, terminations

File: locotouch/assets/go2w_transport/urdf/go2w_transport.urdf (robot description, URDF)
Before this commit: robot go2w_description, 34 links, 33 joints
Links:
- removed link pingban
- added link platform, mass 0.28285; collision mesh filename=../dae/platform.STL; visual mesh filename=../dae/platform.STL
Joints:
- removed joint pingban_to_base
- added joint platform_to_base: type fixed, parent base, child platform, origin xyz=-0.18 -0.107 0.32 rpy=0 1.5708 0

Commit message: add inertia events

File: locotouch/assets/go2w_transport/urdf/go2w_transport.urdf (robot description, URDF)
Before this commit: robot go2w_description, 34 links, 33 joints
Links:
- link platform: geometry collision mesh filename=../dae/platform.STL scale=0.001 0.001 0.001; visual mesh filename=../dae/platform.STL scale=0.001 0.001 0.001
Joints:
- joint platform_to_base: origin xyz=-0.18 -0.107 0.32 rpy=0 1.5708 0 -> xyz=-0.18 -0.107 0.3365 rpy=0 1.5708 0
